File: hardware/split60_ortho/split60_ortho.kicad_sch (KiCad schematic)
At the start: 0 parts

Commit message: Revise layout to split 60
Other:
- title: lily58_ortho_split -> split60_ortho
Changed lines of the file:
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@@
   (paper "A4")
   (title_block
-    (title "lily58_ortho_split")
-    (comment 1 "58-key split keyboard, Pro Micro compatible, TRRS, MX hotswap")
+    (title "split60_ortho")
+    (comment 1 "60-key split keyboard, Pro Micro compatible, TRRS, MX hotswap")
     (comment 2 "Initial schematic placeholder")
   )
